File: pcb/surfboard.kicad_pcb (KiCad board)
At the start: 2 copper layers, 64.3 x 45.2 mm, 24 parts, among them SW1 SW_PUSH, SW2 SW_PUSH, SW3 SW_PUSH, SW4 SW_PUSH, SW5 SW_PUSH, SW6 SW_PUSH, SW7 SW_PUSH, U1 ProMicro

Commit message: Add scissors icons and bump version
Parts:
- added G***: LOGO, phi-kbd-library:Icon-Scissors, B.Cu at (93.8, 50.2)
- added G***: LOGO, phi-kbd-library:Icon-Scissors, B.Cu at (87.2, 52.9)
Other:
- board text added: "hifumi keyboard v1.0 by riconken"
- board text removed: "hifumi keyboard v0.1 by riconken"

Commit message: Slightly move the scissor icons
Parts:
- moved G*** 0.42 mm to (87.5, 52.6)
Changed lines of the file:
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@@
   )
   (module phi-kbd-library:Icon-Scissors (layer B.Cu)
-    (at 87.248362 52.911424 270)
+    (at 87.54602 52.613766 270)
     (fp_text reference G*** (at 0 0 270) (layer B.SilkS) hide
       (effects (font (size 1.524 1.524) (thickness 0.3)) (justify mirror))
